File: pcbs/phy-module-10-base-t1s-v1/eth-conn-cdn.kicad_sch (KiCad schematic)
At the start: 9 parts, among them J201 JST-GH-2-Vertical, J202 JST-GH-2-Vertical

Commit message: [10base-t1s] Updated schematic symbols
Parts:
- J201, J202: symbol JST-GH:JST-GH-2-Vertical -> JST:JST-GH-2-Vertical
Changed lines of the file:
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@@
 	)
 	(symbol
-		(lib_id "JST-GH:JST-GH-2-Vertical")
+		(lib_id "JST:JST-GH-2-Vertical")
 		(at 50.8 91.44 0)
 		(unit 1)
@@
 	)
 	(symbol
-		(lib_id "JST-GH:JST-GH-2-Vertical")
+		(lib_id "JST:JST-GH-2-Vertical")
 		(at 50.8 76.2 0)
 		(unit 1)
