File: pcbs/phy-module-10-base-t1s-v1/microcontroller.kicad_sch (KiCad schematic)
At the start: 20 parts, among them Q601 DMN21D2UFB-7B, U601 STM32L021F4Ux

Commit message: [10base-t1s] Updated schematic symbols
Parts:
- D601, D602, D603: symbol Device:LED_Small -> DEV:LED_SMALL
Changed lines of the file:
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@@
 	)
 	(symbol
-		(lib_id "Device:LED_Small")
+		(lib_id "DEV:LED_SMALL")
 		(at 83.82 154.94 90)
 		(unit 1)
@@
 			)
 		)
+		(property "Sim.Pins" "1=K 2=A"
+			(at 83.82 154.94 0)
+			(effects
+				(font
+					(size 1.27 1.27)
+				)
+				(hide yes)
+			)
+		)
 		(pin "1"
 		)
@@
 	)
 	(symbol
-		(lib_id "Device:LED_Small")
+		(lib_id "DEV:LED_SMALL")
 		(at 114.3 154.94 90)
 		(unit 1)
@@
 		)
 		(property "Sim.Pin" "1=K 2=A"
+			(at 114.3 154.94 0)
+			(effects
+				(font
+					(size 1.27 1.27)
+				)
+				(hide yes)
+			)
+		)
+		(property "Sim.Pins" "1=K 2=A"
 			(at 114.3 154.94 0)
 			(effects
@@
 	)
 	(symbol
-		(lib_id "Device:LED_Small")
+		(lib_id "DEV:LED_SMALL")
 		(at 53.34 154.94 90)
 		(unit 1)
@@
 			(at 53.34 154.94 0)
 			(effects
+				(font
+					(size 1.27 1.27)
+				)
+				(hide yes)
+			)
+		)
+		(property "Sim.Pins" "1=K 2=A"
+			(at 53.34 154.94 0)
+			(effects

Commit message: [10base-t1s-v1] Updated LED footprints
Parts:
- D601, D602, D603: footprint project_footprints:R_0402 -> project_footprints:LED_0402
Changed lines of the file:
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@@
 			)
 		)
-		(property "Footprint" "project_footprints:R_0402"
+		(property "Footprint" "project_footprints:LED_0402"
 			(at 83.82 154.94 90)
 			(hide yes)
@@
 			)
 		)
-		(property "Footprint" "project_footprints:R_0402"
+		(property "Footprint" "project_footprints:LED_0402"
 			(at 114.3 154.94 90)
 			(hide yes)
@@
 			)
 		)
-		(property "Footprint" "project_footprints:R_0402"
+		(property "Footprint" "project_footprints:LED_0402"
 			(at 53.34 154.94 90)
 			(hide yes)
