File: pcbs/term-10base-t1s-v1/term-10base-t1s-v1.kicad_pcb (KiCad board)
At the start: 2 copper layers, 10 x 6 mm, 5 parts

Commit message: [term-10base-t1s] Shrunk to 8mm * 6mm
Parts:
- moved TP1 0.17 mm to (151.5, 98.5)
Routing:
- net Net-(R2-Pad2): track 0.00 -> 2.87 mm
- net Net-(R1-Pad1): track 0.00 -> 2.87 mm
- net Net-(C1-Pad2): track 0.00 -> 1.01 mm
- net Net-(C1-Pad1): track 0.00 -> 1.01 mm
Other:
- board size 10 x 6 mm -> 8 x 6 mm
